Commit message: Basic kitchen counter demo - objects in cabinets

File: exploration/PRPL_lab/urdf/PRPL_lab_collision.urdf (robot description, URDF)
Before this commit: robot PRPL_lab, 62 links, 61 joints
Links:
- link Baseboard2.001_link: geometry visual mesh filename=../meshes/stl/Baseboard2.001.stl scale=1.00000 1.00000 1.00000
- link Cabinet1.001_link: geometry visual mesh filename=../meshes/stl/Cabinet1.005.stl scale=1.00000 1.00000 1.00000
- link Cabinet1.002_link: geometry visual mesh filename=../meshes/stl/Cabinet1.002.stl scale=1.00000 1.00000 1.00000
- link Cabinet1.003_link: geometry visual mesh filename=../meshes/stl/Cabinet1.009.stl scale=1.00000 1.00000 1.00000
- link Cabinet1.004_link: geometry visual mesh filename=../meshes/stl/Cabinet1.003.stl scale=1.00000 1.00000 1.00000
- link Cabinet1.007_link: geometry visual mesh filename=../meshes/stl/Cabinet1.001.stl scale=1.00000 1.00000 1.00000
- link Cabinet1_Door.001_link: geometry visual mesh filename=../meshes/stl/Cabinet1_Door.004.stl scale=1.00000 1.00000 1.00000
- link Cabinet1_Door.002_link: geometry visual mesh filename=../meshes/stl/Cabinet1_Door.002.stl scale=1.00000 1.00000 1.00000
- link Cabinet1_Door.003_link: geometry visual mesh filename=../meshes/stl/Cabinet1_Door.001.stl scale=1.00000 1.00000 1.00000
- link Cabinet1_Door.004_link: geometry visual mesh filename=../meshes/stl/Cabinet1_Door.005.stl scale=1.00000 1.00000 1.00000
- link Cabinet1_Door.005_link: geometry visual mesh filename=../meshes/stl/Cabinet1_Door.008.stl scale=1.00000 1.00000 1.00000
- link Cabinet1_Door.006_link: geometry visual mesh filename=../meshes/stl/Cabinet1_Door.006.stl scale=1.00000 1.00000 1.00000
- link Cabinet1_Door_link: geometry visual mesh filename=../meshes/stl/Cabinet1_Door.003.stl scale=1.00000 1.00000 1.00000
- link Cabinet1_link: geometry visual mesh filename=../meshes/stl/Cabinet1.004.stl scale=1.00000 1.00000 1.00000
- link Cabinet2_Door.001_link: geometry visual mesh filename=../meshes/stl/Cabinet2_Door.003.stl scale=1.00000 1.00000 1.00000
- link Cabinet2_Door.002_link: geometry visual mesh filename=../meshes/stl/Cabinet2_Door.001.stl scale=1.00000 1.00000 1.00000
- link Cabinet2_Door.003_link: geometry visual mesh filename=../meshes/stl/Cabinet2_Door.005.stl scale=1.00000 1.00000 1.00000
- link Cabinet2_Door.004_link: geometry visual mesh filename=../meshes/stl/Cabinet2_Door.007.stl scale=1.00000 1.00000 1.00000
- link Cabinet2_Door.005_link: geometry visual mesh filename=../meshes/stl/Cabinet2_Door.004.stl scale=1.00000 1.00000 1.00000
- link Cabinet2_Door_link: geometry visual mesh filename=../meshes/stl/Cabinet2_Door.002.stl scale=1.00000 1.00000 1.00000
- link Drawer.001_link: geometry visual mesh filename=../meshes/stl/Drawer.004.stl scale=1.00000 1.00000 1.00000
- link Drawer.002_link: geometry visual mesh filename=../meshes/stl/Drawer.005.stl scale=1.00000 1.00000 1.00000
- link Drawer.003_link: geometry visual mesh filename=../meshes/stl/Drawer.012.stl scale=1.00000 1.00000 1.00000
- link Drawer.004_link: geometry visual mesh filename=../meshes/stl/Drawer.013.stl scale=1.00000 1.00000 1.00000
- link Drawer.005_link: geometry visual mesh filename=../meshes/stl/Drawer.014.stl scale=1.00000 1.00000 1.00000
- link Drawer_link: geometry visual mesh filename=../meshes/stl/Drawer.003.stl scale=1.00000 1.00000 1.00000
- link Handle.001_link: geometry visual mesh filename=../meshes/stl/Handle.004.stl scale=1.00000 1.00000 1.00000
- link Handle.002_link: geometry visual mesh filename=../meshes/stl/Handle.005.stl scale=1.00000 1.00000 1.00000
- link Handle.003_link: geometry visual mesh filename=../meshes/stl/Handle.002.stl scale=1.00000 1.00000 1.00000
- link Handle.004_link: geometry visual mesh filename=../meshes/stl/Handle.003.stl scale=1.00000 1.00000 1.00000
- link Handle.005_link: geometry visual mesh filename=../meshes/stl/Handle.006.stl scale=1.00000 1.00000 1.00000
- link Handle.006_link: geometry visual mesh filename=../meshes/stl/Handle.007.stl scale=1.00000 1.00000 1.00000
- link Handle.007_link: geometry visual mesh filename=../meshes/stl/Handle.011.stl scale=1.00000 1.00000 1.00000
- link Handle.008_link: geometry visual mesh filename=../meshes/stl/Handle.012.stl scale=1.00000 1.00000 1.00000
- link Handle.012_link: geometry visual mesh filename=../meshes/stl/Handle.009.stl scale=1.00000 1.00000 1.00000
- link Handle.013_link: geometry visual mesh filename=../meshes/stl/Handle.010.stl scale=1.00000 1.00000 1.00000
- link Handle_link: geometry visual mesh filename=../meshes/stl/Handle.008.stl scale=1.00000 1.00000 1.00000
